File: Heatpump_controller.kicad_sch (KiCad schematic)
At the start: 45 parts, among them J1 Conn_01x03, J2 USB_C_Receptacle_USB2.0_16P, J3 Conn_01x03, J4 Conn_01x03, J5 RJ12, J6 RJ12, K1 SANYOU_SRD_Form_C, K2 SANYOU_SRD_Form_C, K3 SANYOU_SRD_Form_C, Q1 AO3400A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

Commit message: Finished route
Parts:
- added C25, C26: 100nF, Capacitor_SMD:C_0603_1608Metric, symbol Device:C
- added H1, H2, H3, H4: MountingHole, MountingHole:MountingHole_3.2mm_M3, symbol Mechanical:MountingHole
Connections:
- net +3.3V: now also C26.2
- net +5V: now also C25.2
- net GND: now also C25.1, C26.1
- net at Q1.1 (G), R1.1: now also U1.8 (IO32); no longer U1.24 (IO2)
- net at Q2.1 (G), R2.1: now also U1.24 (IO2); no longer U1.26 (IO4)
- net at Q3.1 (G), R3.1: now also U1.26 (IO4); no longer U1.8 (IO32)
Other:
- added sheet Power (Power.kicad_sch)

Commit message: Added lcsc power numbers
Parts:
- C1, C2, C25, C26: LCSC (none) -> C14663
- C15, C16: LCSC (none) -> C15850
- C17: LCSC (none) -> C28323
- D1, D2, D3: LCSC (none) -> C2128
- D4: LCSC (none) -> C2297
- Q1, Q2, Q3: LCSC (none) -> C20917
- Q4, Q5: LCSC (none) -> C2150
- R1, R2, R3, R30: LCSC (none) -> C25804
- R25, R26: LCSC (none) -> C23186
- R27, R28: LCSC (none) -> C22790
- R29: LCSC (none) -> C22859
- R31: LCSC (none) -> C21190
- R4, R8: LCSC (none) -> C22775
- R5, R6, R7, R9: LCSC (none) -> C23162
- U1: LCSC (none) -> C701342
- U2: LCSC (none) -> C3035748
- U3, U4: LCSC (none) -> C8963
