File: Power.kicad_sch (KiCad schematic)
At the start: 13 parts, among them U6 TPS54331

Commit message: Added lcsc power numbers
Parts:
- C18, C19: LCSC (none) -> C15850
- C20: LCSC (none) -> C1322360
- C21: LCSC (none) -> C1634
- C22: LCSC (none) -> C1628
- C23: LCSC (none) -> C14663
- C24: LCSC (none) -> C16780
- D5: LCSC (none) -> C8678
- U6: LCSC (none) -> C9865
Changed lines of the file:
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@@
+			)
+		)
+		(property "LCSC" "C15850"
+			(at 116.205 85.725 0)
+			(effects
+				(font
+					(size 1.27 1.27)
+				)
+				(hide yes)
 			)
 		)
@@
 		)
 		(property "Description" "Unpolarized capacitor"
+			(at 120.65 100.33 0)
+			(effects
+				(font
+					(size 1.27 1.27)
+				)
+				(hide yes)
+			)
+		)
+		(property "LCSC" "C1322360"
 			(at 120.65 100.33 0)
 			(effects
@@
 			)
 		)
+		(property "LCSC" "C9865"
+			(at 158.75 85.725 0)
+			(effects
+				(font
+					(size 1.27 1.27)
+				)
+				(hide yes)
+			)
+		)
 		(pin "5"
 		)
@@
 			)
 		)
+		(property "LCSC" "C15850"
+			(at 104.775 85.725 0)
+			(effects
+				(font
+					(size 1.27 1.27)
+				)
+				(hide yes)
+			)
+		)
 		(pin "1"
 		)
@@
 		)
 		(property "Description" "Unpolarized capacitor"
+			(at 127.635 100.33 0)
+			(effects
+				(font
+					(size 1.27 1.27)
+				)
+				(hide yes)
+			)
+		)
+		(property "LCSC" "C1634"
 			(at 127.635 100.33 0)
 			(effects
@@
 			)
 		)
+		(property "LCSC" "C16780"
+			(at 201.93 91.44 0)
+			(effects
+				(font
+					(size 1.27 1.27)
+				)
+				(hide yes)
+			)
+		)
 		(pin "1"
 		)
@@
 			)
 		)
+		(property "LCSC" "C1628"
+			(at 140.97 111.125 0)
+			(effects
+				(font
+					(size 1.27 1.27)
+				)
+				(hide yes)
+			)
+		)
 		(pin "1"
 		)
@@
 		)
 		(property "Description" "Unpolarized capacitor"
+			(at 173.355 81.915 0)
+			(effects
+				(font
+					(size 1.27 1.27)
+				)
+				(hide yes)
+			)
+		)
+		(property "LCSC" "C14663"
 			(at 173.355 81.915 0)
 			(effects
@@
 			(effects
 				(font
+					(size 1.27 1.27)
+				)
+				(hide yes)
+			)
+		)
+		(property "LCSC" "C8678"
+			(at 178.435 92.075 90)
+			(effects
+				(font
